File: Hardware/DoorBellRepeater.sch (EAGLE design)
At the start: 25 parts, among them IC1 LM1117

Commit message: Add files via upload
Parts:
- added LSP1, LSP2: LSP10, solpad:LSP10
Connections:
- new net N$2: HLK-PM01-5V.AC2, LSP1.MP
- net N$6: now also LSP2.MP; no longer HLK-PM01-5V.AC2
Other:
- note added: "Fuse"
Changed lines of the file:
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@@
 <part name="C3" library="adafruit" deviceset="C-US" device="C0805K" value="100uF"/>
 <part name="GND7" library="supply1" library_urn="urn:adsk.eagle:library:371" deviceset="GND" device=""/>
+<part name="LSP1" library="solpad" library_urn="urn:adsk.eagle:library:364" deviceset="LSP10" device="" package3d_urn="urn:adsk.eagle:package:26501/1"/>
+<part name="LSP2" library="solpad" library_urn="urn:adsk.eagle:library:364" deviceset="LSP10" device="" package3d_urn="urn:adsk.eagle:package:26501/1"/>
 </parts>
 <sheets>
@@
 TX
 RX</text>
+<text x="-104.14" y="81.28" size="1.778" layer="91">Fuse</text>
 </plain>
 <instances>
@@
 <instance part="GND7" gate="1" x="-99.06" y="17.78" smashed="yes">
 <attribute name="VALUE" x="-101.6" y="15.24" size="1.778" layer="96"/>
+</instance>
+<instance part="LSP1" gate="1" x="-99.06" y="76.2" smashed="yes" rot="R90">
+<attribute name="NAME" x="-101.981" y="74.93" size="1.778" layer="95" rot="R90"/>
+</instance>
+<instance part="LSP2" gate="1" x="-106.68" y="76.2" smashed="yes" rot="R270">
+<attribute name="NAME" x="-103.759" y="77.47" size="1.778" layer="95" rot="R270"/>
 </instance>
 </instances>
@@
 <segment>
 <pinref part="E1" gate="P" pin="P"/>
+<wire x1="-114.3" y1="76.2" x2="-109.22" y2="76.2" width="0.1524" layer="91"/>
+<pinref part="LSP2" gate="1" pin="MP"/>
+</segment>
+</net>
+<net name="N$2" class="0">
+<segment>
 <pinref part="HLK-PM01-5V" gate="G$1" pin="AC2"/>
-<wire x1="-114.3" y1="76.2" x2="-93.98" y2="76.2" width="0.1524" layer="91"/>
-</segment>
-</net>
+<pinref part="LSP1" gate="1" pin="MP"/>
+<wire x1="-96.52" y1="76.2" x2="-93.98" y2="76.2" width="0.1524" layer="91"/>
+</segment>
+</net>
